Commit message: bora de X?

File: resources/robots/guaraci/urdf/guaraci.urdf (robot description, URDF)
Before this commit: robot guaraci, 25 links, 24 joints
Links:
- link base: geometry collision mesh filename=../meshes/body100.dae scale=0.001 0.001 0.001; visual mesh filename=../meshes/body100.dae scale=0.001 0.001 0.001
- link coxa_l1: geometry collision mesh filename=../meshes/coxa.dae scale=0.001 0.001 0.001; visual mesh filename=../meshes/coxa.dae scale=0.001 0.001 0.001
- link coxa_l2: geometry collision mesh filename=../meshes/coxa.dae scale=0.001 0.001 0.001; visual mesh filename=../meshes/coxa.dae scale=0.001 0.001 0.001
- link coxa_l3: geometry collision mesh filename=../meshes/coxa.dae scale=0.001 0.001 0.001; visual mesh filename=../meshes/coxa.dae scale=0.001 0.001 0.001
- link coxa_r1: geometry collision mesh filename=../meshes/coxa.dae scale=0.001 0.001 0.001; visual mesh filename=../meshes/coxa.dae scale=0.001 0.001 0.001
- link coxa_r2: geometry collision mesh filename=../meshes/coxa.dae scale=0.001 0.001 0.001; visual mesh filename=../meshes/coxa.dae scale=0.001 0.001 0.001
- link coxa_r3: geometry collision mesh filename=../meshes/coxa.dae scale=0.001 0.001 0.001; visual mesh filename=../meshes/coxa.dae scale=0.001 0.001 0.001
- link femur_l1: geometry collision mesh filename=../meshes/femur220.dae scale=0.001 0.001 0.001; visual mesh filename=../meshes/femur220.dae scale=0.001 0.001 0.001
- link femur_l2: geometry collision mesh filename=../meshes/femur220.dae scale=0.001 0.001 0.001; visual mesh filename=../meshes/femur220.dae scale=0.001 0.001 0.001
- link femur_l3: geometry collision mesh filename=../meshes/femur220.dae scale=0.001 0.001 0.001; visual mesh filename=../meshes/femur220.dae scale=0.001 0.001 0.001
- link femur_r1: geometry collision mesh filename=../meshes/femur220.dae scale=0.001 0.001 0.001; visual mesh filename=../meshes/femur220.dae scale=0.001 0.001 0.001
- link femur_r2: geometry collision mesh filename=../meshes/femur220.dae scale=0.001 0.001 0.001; visual mesh filename=../meshes/femur220.dae scale=0.001 0.001 0.001
- link femur_r3: geometry collision mesh filename=../meshes/femur220.dae scale=0.001 0.001 0.001; visual mesh filename=../meshes/femur220.dae scale=0.001 0.001 0.001
- link foot_l1: geometry collision mesh filename=../meshes/foot.dae scale=0.001 0.001 0.001; visual mesh filename=../meshes/foot.dae scale=0.001 0.001 0.001
- link foot_l2: geometry collision mesh filename=../meshes/foot.dae scale=0.001 0.001 0.001; visual mesh filename=../meshes/foot.dae scale=0.001 0.001 0.001
- link foot_l3: geometry collision mesh filename=../meshes/foot.dae scale=0.001 0.001 0.001; visual mesh filename=../meshes/foot.dae scale=0.001 0.001 0.001
- link foot_r1: geometry collision mesh filename=../meshes/foot.dae scale=0.001 0.001 0.001; visual mesh filename=../meshes/foot.dae scale=0.001 0.001 0.001
- link foot_r2: geometry collision mesh filename=../meshes/foot.dae scale=0.001 0.001 0.001; visual mesh filename=../meshes/foot.dae scale=0.001 0.001 0.001
- link foot_r3: geometry collision mesh filename=../meshes/foot.dae scale=0.001 0.001 0.001; visual mesh filename=../meshes/foot.dae scale=0.001 0.001 0.001
- link tibia_l1: geometry collision mesh filename=../meshes/tibia_3.dae scale=0.001 0.001 0.001; visual mesh filename=../meshes/tibia_3.dae scale=0.001 0.001 0.001
- link tibia_l2: geometry collision mesh filename=../meshes/tibia_3.dae scale=0.001 0.001 0.001; visual mesh filename=../meshes/tibia_3.dae scale=0.001 0.001 0.001
- link tibia_l3: geometry collision mesh filename=../meshes/tibia_3.dae scale=0.001 0.001 0.001; visual mesh filename=../meshes/tibia_3.dae scale=0.001 0.001 0.001
- link tibia_r1: geometry collision mesh filename=../meshes/tibia_3.dae scale=0.001 0.001 0.001; visual mesh filename=../meshes/tibia_3.dae scale=0.001 0.001 0.001
- link tibia_r2: geometry collision mesh filename=../meshes/tibia_3.dae scale=0.001 0.001 0.001; visual mesh filename=../meshes/tibia_3.dae scale=0.001 0.001 0.001
- link tibia_r3: geometry collision mesh filename=../meshes/tibia_3.dae scale=0.001 0.001 0.001; visual mesh filename=../meshes/tibia_3.dae scale=0.001 0.001 0.001

Commit message: fist train success

File: resources/robots/guaraci/urdf/guaraci.urdf (robot description, URDF)
Before this commit: robot guaraci, 25 links, 24 joints
Links:
- removed link foot_l1
- removed link foot_l2
- removed link foot_l3
- removed link foot_r1
- removed link foot_r2
- removed link foot_r3
- added link l1_FOOT, mass 1.15784; collision sphere radius=0.03; visual mesh filename=../meshes/foot.dae scale=0.001 0.001 0.001
- added link l2_FOOT, mass 1.15784; collision sphere radius=0.03; visual mesh filename=../meshes/foot.dae scale=0.001 0.001 0.001
- added link l3_FOOT, mass 1.15784; collision sphere radius=0.03; visual mesh filename=../meshes/foot.dae scale=0.001 0.001 0.001
- added link r1_FOOT, mass 1.15784; collision sphere radius=0.03; visual mesh filename=../meshes/foot.dae scale=0.001 0.001 0.001
- added link r2_FOOT, mass 1.15784; collision sphere radius=0.03; visual mesh filename=../meshes/foot.dae scale=0.001 0.001 0.001
- added link r3_FOOT, mass 1.15784; collision sphere radius=0.03; visual mesh filename=../meshes/foot.dae scale=0.001 0.001 0.001
- link tibia_l1: geometry visual mesh filename=../meshes/tibia_3.dae scale=0.001 0.001 0.001
- link tibia_l2: geometry visual mesh filename=../meshes/tibia_3.dae scale=0.001 0.001 0.001
- link tibia_l3: geometry visual mesh filename=../meshes/tibia_3.dae scale=0.001 0.001 0.001
- link tibia_r1: geometry visual mesh filename=../meshes/tibia_3.dae scale=0.001 0.001 0.001
- link tibia_r2: geometry visual mesh filename=../meshes/tibia_3.dae scale=0.001 0.001 0.001
- link tibia_r3: geometry visual mesh filename=../meshes/tibia_3.dae scale=0.001 0.001 0.001
Joints:
- removed joint joint_foot_l1
- removed joint joint_foot_l2
- removed joint joint_foot_l3
- removed joint joint_foot_r1
- removed joint joint_foot_r2
- removed joint joint_foot_r3
- added joint joint_l1_FOOT: type fixed, parent tibia_l1, child l1_FOOT, origin xyz=0.19859 0 0 rpy=1.5707 0 0
- added joint joint_l2_FOOT: type fixed, parent tibia_l2, child l2_FOOT, origin xyz=0.19859 0 0 rpy=1.5707 0 0
- added joint joint_l3_FOOT: type fixed, parent tibia_l3, child l3_FOOT, origin xyz=0.19859 0 0 rpy=1.5707 0 0
- added joint joint_r1_FOOT: type fixed, parent tibia_r1, child r1_FOOT, origin xyz=0.19859 0 0 rpy=1.5707 0 0
- added joint joint_r2_FOOT: type fixed, parent tibia_r2, child r2_FOOT, origin xyz=0.19859 0 0 rpy=1.5707 0 0
- added joint joint_r3_FOOT: type fixed, parent tibia_r3, child r3_FOOT, origin xyz=0.19859 0 0 rpy=1.5707 0 0
- joint joint_coxa_l1: limit lower=-3.14159 upper=3.14159 effort=25.0 velocity=0.5 -> lower=-3.14159 upper=3.14159 effort=80.0 velocity=20.0; origin xyz=0.17302 -0.10517 0 rpy=3.14159 0 5.4977 -> xyz=0.17302 -0.10517 0 rpy=3.14159 0 7.0684
- joint joint_coxa_l2: limit lower=-3.14159 upper=3.14159 effort=25.0 velocity=0.5 -> lower=-3.14159 upper=3.14159 effort=80.0 velocity=20.0; origin xyz=0 -0.169 0 rpy=3.14159 0 4.71229 -> xyz=0 -0.169 0 rpy=3.14159 0 6.28299
- joint joint_coxa_l3: limit lower=-3.14159 upper=3.14159 effort=25.0 velocity=0.5 -> lower=-3.14159 upper=3.14159 effort=80.0 velocity=20.0; origin xyz=-0.17302 -0.10517 0 rpy=3.14159 0 3.9269 -> xyz=-0.17302 -0.10517 0 rpy=3.14159 0 5.4976
- joint joint_coxa_r1: limit lower=-3.14159 upper=3.14159 effort=25.0 velocity=0.5 -> lower=-3.14159 upper=3.14159 effort=80.0 velocity=20.0; origin xyz=0.17302 0.10517 0 rpy=3.14159 0 0.7854 -> xyz=0.17302 0.10517 0 rpy=3.14159 0 2.35605
- joint joint_coxa_r2: limit lower=-3.14159 upper=3.14159 effort=25.0 velocity=0.5 -> lower=-3.14159 upper=3.14159 effort=80.0 velocity=20.0; origin xyz=0 0.169 0 rpy=3.14159 0 1.5707 -> xyz=0 0.169 0 rpy=3.14159 0 3.14159
- joint joint_coxa_r3: limit lower=-3.14159 upper=3.14159 effort=25.0 velocity=0.5 -> lower=-3.14159 upper=3.14159 effort=80.0 velocity=20.0; origin xyz=-0.17302 0.10517 0 rpy=3.14159 0 2.3561 -> xyz=-0.17302 0.10517 0 rpy=3.14159 0 3.92694
- joint joint_femur_l1: limit lower=-3.14159 upper=3.14159 effort=25.0 velocity=0.5 -> lower=-3.14159 upper=3.14159 effort=80.0 velocity=20.0; origin xyz=0.09041 0 0 rpy=1.5707 0 0 -> xyz=0 0.09041 0 rpy=1.5707 0 1.5707
- joint joint_femur_l2: limit lower=-3.14159 upper=3.14159 effort=25.0 velocity=0.5 -> lower=-3.14159 upper=3.14159 effort=80.0 velocity=20.0; origin xyz=0.09041 0 0 rpy=1.5707 0 0 -> xyz=0 0.09041 0 rpy=1.5707 0 1.5707
- joint joint_femur_l3: limit lower=-3.14159 upper=3.14159 effort=25.0 velocity=0.5 -> lower=-3.14159 upper=3.14159 effort=80.0 velocity=20.0; origin xyz=0.09041 0 0 rpy=1.5707 0 0 -> xyz=0 0.09041 0 rpy=1.5707 0 1.5707
- joint joint_femur_r1: limit lower=-3.14159 upper=3.14159 effort=25.0 velocity=0.5 -> lower=-3.14159 upper=3.14159 effort=80.0 velocity=20.0; origin xyz=0.09041 0 0 rpy=1.5707 0 0 -> xyz=0 0.09041 0 rpy=1.5707 0 1.5707
- joint joint_femur_r2: limit lower=-3.14159 upper=3.14159 effort=25.0 velocity=0.5 -> lower=-3.14159 upper=3.14159 effort=80.0 velocity=20.0; origin xyz=0.09041 0 0 rpy=1.5707 0 0 -> xyz=0 0.09041 0 rpy=1.5707 0 1.5707
- joint joint_femur_r3: limit lower=-3.14159 upper=3.14159 effort=25.0 velocity=0.5 -> lower=-3.14159 upper=3.14159 effort=80.0 velocity=20.0; origin xyz=0.09041 0 0 rpy=1.5707 0 0 -> xyz=0 0.09041 0 rpy=1.5707 0 1.5707
- joint joint_tibia_l1: limit lower=-3.14159 upper=3.14159 effort=25.0 velocity=0.5 -> lower=-3.14159 upper=3.14159 effort=80.0 velocity=20.0
- joint joint_tibia_l2: limit lower=-3.14159 upper=3.14159 effort=25.0 velocity=0.5 -> lower=-3.14159 upper=3.14159 effort=80.0 velocity=20.0
- joint joint_tibia_l3: limit lower=-3.14159 upper=3.14159 effort=25.0 velocity=0.5 -> lower=-3.14159 upper=3.14159 effort=80.0 velocity=20.0
- joint joint_tibia_r1: limit lower=-3.14159 upper=3.14159 effort=25.0 velocity=0.5 -> lower=-3.14159 upper=3.14159 effort=80.0 velocity=20.0
- joint joint_tibia_r2: limit lower=-3.14159 upper=3.14159 effort=25.0 velocity=0.5 -> lower=-3.14159 upper=3.14159 effort=80.0 velocity=20.0
- joint joint_tibia_r3: limit lower=-3.14159 upper=3.14159 effort=25.0 velocity=0.5 -> lower=-3.14159 upper=3.14159 effort=80.0 velocity=20.0

Commit message: new tibia

File: resources/robots/guaraci/urdf/guaraci.urdf (robot description, URDF)
Before this commit: robot guaraci, 25 links, 24 joints
Links:
- link base: mass 9.42278 -> 16.2
- link coxa_l1: mass 0.59759 -> 1.655
- link coxa_l2: mass 0.59759 -> 1.655
- link coxa_l3: mass 0.59759 -> 1.655
- link coxa_r1: mass 0.59759 -> 1.655
- link coxa_r2: mass 0.59759 -> 1.655
- link coxa_r3: mass 0.59759 -> 1.655
- link l1_FOOT: mass 1.15784 -> 0.2
- link l2_FOOT: mass 1.15784 -> 0.2
- link l3_FOOT: mass 1.15784 -> 0.2
- link r1_FOOT: mass 1.15784 -> 0.2
- link r2_FOOT: mass 1.15784 -> 0.2
- link r3_FOOT: mass 1.15784 -> 0.2
- link tibia_l1: mass 0.71403 -> 1.455; geometry visual mesh filename=../meshes/tibia_393.stl scale=0.001 0.001 0.001
- link tibia_l2: mass 0.71403 -> 1.455; geometry visual mesh filename=../meshes/tibia_393.stl scale=0.001 0.001 0.001
- link tibia_l3: mass 0.71403 -> 1.455; geometry visual mesh filename=../meshes/tibia_393.stl scale=0.001 0.001 0.001
- link tibia_r1: mass 0.71403 -> 1.455; geometry visual mesh filename=../meshes/tibia_393.stl scale=0.001 0.001 0.001
- link tibia_r2: mass 0.71403 -> 1.455; geometry visual mesh filename=../meshes/tibia_393.stl scale=0.001 0.001 0.001
- link tibia_r3: mass 0.71403 -> 1.455; geometry visual mesh filename=../meshes/tibia_393.stl scale=0.001 0.001 0.001
Joints:
- joint joint_l1_FOOT: origin xyz=0.19859 0 0 rpy=1.5707 0 0 -> xyz=0.36734 0 0 rpy=1.5707 0 0
- joint joint_l2_FOOT: origin xyz=0.19859 0 0 rpy=1.5707 0 0 -> xyz=0.36734 0 0 rpy=1.5707 0 0
- joint joint_l3_FOOT: origin xyz=0.19859 0 0 rpy=1.5707 0 0 -> xyz=0.36734 0 0 rpy=1.5707 0 0
- joint joint_r1_FOOT: origin xyz=0.19859 0 0 rpy=1.5707 0 0 -> xyz=0.36734 0 0 rpy=1.5707 0 0
- joint joint_r2_FOOT: origin xyz=0.19859 0 0 rpy=1.5707 0 0 -> xyz=0.36734 0 0 rpy=1.5707 0 0
- joint joint_r3_FOOT: origin xyz=0.19859 0 0 rpy=1.5707 0 0 -> xyz=0.36734 0 0 rpy=1.5707 0 0
